File: PLC4UNI-GC1_PCB/_restore_backup_2026-07-14T23-10-33-515/PLC4UNI-GC1.kicad_pcb (KiCad board)
At the start: 4 copper layers, 102.4 x 83.1 mm, 179 parts, among them J1 Conn_02x08_Odd_Even, K1 G5V-1, K2 G5V-1, Q1 NCE60P04R, Q2 ZXMS6004FFQTA, Q3 ZXMS6004FFQTA, Q4 ZXMS6004FFQTA, Q5 ZXMS6004FFQTA, SW1 TS-1088-AR02016, U1 ESP32-S3-WROOM-1, U10 ADS1115IDGS, U11 AT3H4B-CUH-S, U12 AT3H4B-CUH-S, U13 LK1802, U14 AT3H4B-CUH-S, U15 MAX31856MUD+, U16 BL0942, U17 B0303S-1WR3_C7465185, U18 ISO7021DR, U2 AT3H4B-CUH-S, U3 AP63203WU, U4 RS485-PROTECT, U5 AT3H4B-CUH-S, U6 AT3H4B-CUH-S, U7 GP8211S-TC50-EW, U8 GP8302-TC50-EW, U9 BTS723GWXUMA1

Commit message: edge.cuts update
areglo d e cortes de placa estaban desalineados
Parts:
- moved C19 34.5 mm to (161.4, 93.2), turned to 180 degrees
- moved R43 14.1 mm to (143.1, 85.3)
- moved C34 6.42 mm to (161.9, 80.5), turned to 0 degrees
- moved C33 5.84 mm to (161.9, 84.6), turned to 0 degrees
- moved D14 4.85 mm to (151.5, 80.0)
- moved TP4 4.54 mm to (151.5, 82.8)
- moved R48 4.21 mm to (161.9, 78.5), turned to 0 degrees
- moved D16 3.60 mm to (162.9, 85.6), turned to 0 degrees
- moved D15 3.58 mm to (161.9, 82.5), turned to 0 degrees
- moved D13 3.31 mm to (151.5, 77.2), turned to -90 degrees
- moved R29 3.30 mm to (156.6, 84.4)
- moved R9 3.11 mm to (156.6, 74.7), turned to 0 degrees
- moved C24 2.96 mm to (156.6, 86.6), turned to 180 degrees
- moved C28 2.73 mm to (135.0, 76.4), turned to 180 degrees
- moved R49 2.02 mm to (161.9, 86.6), turned to 0 degrees
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Routing:
- net /control/IN-0-10V1/OUT3V: track 11.4 -> 0.00 mm
- net Net-(D15-K): track 10.7 -> 0.00 mm
- net Net-(D10-K): track 8.34 -> 0.00 mm
- net /control/IN-0-10V/OUT3V: track 15.7 -> 8.67 mm
- net /control/IN-4-20MA/OUT: track 6.99 -> 0.00 mm
- net /control/CON-IN-4-20MA_1: track 5.93 -> 0.00 mm
- net /control/CON-IN-4-20MA_2: track 5.80 -> 0.00 mm
- net /control/CON_IN_0-10V_2: track 5.79 -> 0.00 mm
- net GND: track 31.7 -> 26.4 mm, vias 50 -> 40
- net /control/IN-4-20MA1/OUT: track 4.38 -> 0.00 mm
- net Net-(C12-Pad1): track 4.36 -> 0.00 mm
- net Net-(C33-Pad1): track 4.34 -> 0.00 mm, vias 1 -> 0
- net Net-(U15-~{DRDY}): track 3.73 -> 0.00 mm
- net /control/IN-0-10V1/COM: track 2.90 -> 0.00 mm
- net +3.3V: track 17.7 -> 16.6 mm, vias 20 -> 18
