File: PLC4UNI-GC1_PCB/_restore_backup_2026-07-14T23-10-33-515/PLC4UNI-GC1.kicad_sch (KiCad schematic)
At the start: 6 parts

Commit message: edge.cuts update
areglo d e cortes de placa estaban desalineados
Other:
- removed sheet paul martinez
Changed lines of the file:
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@@
-	)
-	(sheet
-		(at 165.1 50.8)
-		(size 12.7 3.81)
-		(exclude_from_sim no)
-		(in_bom yes)
-		(on_board yes)
-		(dnp no)
-		(fields_autoplaced yes)
-		(stroke
-			(width 0.1524)
-			(type solid)
-		)
-		(fill
-			(color 0 0 0 0)
-		)
-		(property "Sheetname" "paul martinez"
-			(at 165.1 50.0884 0)
-			(show_name no)
-			(do_not_autoplace no)
-			(effects
-				(font
-					(size 1.27 1.27)
-				)
-				(justify left bottom)
-			)
-		)
-		(property "Sheetfile" "paulmartinez.kicad_sch"
-			(at 165.1 55.1946 0)
-			(show_name no)
-			(do_not_autoplace no)
-			(effects
-				(font
-					(size 1.27 1.27)
-				)
-				(justify left top)
-			)
-		)
-		(instances
-			(project "PLC4UNI-GC1"
-				(path "/78be00cd-daf6-4f2a-9977-d3085e20b798"
-					(page "22")
-				)
-			)
-		)
 	)
 	(sheet
