File: PLC4UNI-GC1_PCB/PLC4UNI-GC1.kicad_pcb (KiCad board)
At the start: 4 copper layers, 102.4 x 83.1 mm, 179 parts, among them J1 Conn_02x08_Odd_Even, K1 G5V-1, K2 G5V-1, Q1 NCE60P04R, Q2 ZXMS6004FFQTA, Q3 ZXMS6004FFQTA, Q4 ZXMS6004FFQTA, Q5 ZXMS6004FFQTA, SW1 TS-1088-AR02016, U1 ESP32-S3-WROOM-1, U10 ADS1115IDGS, U11 AT3H4B-CUH-S, U12 AT3H4B-CUH-S, U13 LK1802, U14 AT3H4B-CUH-S, U15 MAX31856MUD+, U16 BL0942, U17 B0303S-1WR3_C7465185, U18 ISO7021DR, U2 AT3H4B-CUH-S, U3 AP63203WU, U4 RS485-PROTECT, U5 AT3H4B-CUH-S, U6 AT3H4B-CUH-S, U7 GP8211S-TC50-EW, U8 GP8302-TC50-EW, U9 BTS723GWXUMA1

Commit message: signals analogical
Parts:
- moved D6 4.29 mm to (94.2, 71.5)
- moved U12 3.18 mm to (120.1, 81.7)
- moved D1 3.03 mm to (90.0, 68.1)
- moved TP7 1.91 mm to (89.9, 63.4)
- moved R23 1.63 mm to (120.9, 71.8)
- moved R21 1.52 mm to (119.1, 71.8)
- moved R20 1.45 mm to (115.0, 86.5)
- moved C18 1.38 mm to (120.1, 76.7), turned to 180 degrees
- moved U6 1.37 mm to (125.5, 80.3)
- moved C16 1.32 mm to (115.0, 75.0)
- moved U11 1.31 mm to (115.1, 79.9)
- moved R3 1.30 mm to (125.4, 86.7), turned to 180 degrees
- moved C20 1.28 mm to (125.4, 85.0)
- moved C17 1.25 mm to (115.0, 84.8)
- moved C3 1.22 mm to (125.5, 74.9)
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Routing:
- net +24V: track 202.1 -> 179.4 mm, vias 5 -> 11
- net /control/IN_NPN4: track 0.00 -> 13.3 mm
- net /PowerSupply/vdc_in: track 39.1 -> 25.9 mm
- net GND: track 31.7 -> 43.1 mm, vias 50 -> 66
- net Net-(C33-Pad1): track 4.34 -> 12.2 mm
- net Net-(C3-Pad1): track 0.00 -> 7.16 mm
- net Net-(C18-Pad1): track 0.00 -> 6.85 mm
- net Net-(C16-Pad1): track 0.00 -> 6.72 mm
- net /control/IN-0-10V1/OUT3V: track 11.4 -> 18.1 mm
- net /control/CON_IN_NPN4: track 0.00 -> 6.17 mm
- net Net-(C14-Pad1): track 0.00 -> 6.04 mm
- net /control/CON_IN_PNP1: track 0.00 -> 5.97 mm
- net /control/CON_IN_NPN3: track 0.00 -> 5.53 mm
- net Net-(C4-Pad1): track 2.46 -> 7.07 mm
- net /control/IN_NPN3: track 0.00 -> 3.68 mm
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- added copper zone on In2.Cu, net +24V

Commit message: Esp32 finish
Parts:
- moved LED5 37.5 mm to (146.0, 116.5)
- moved R50 37.5 mm to (143.4, 116.4)
- moved TP6 7.26 mm to (88.7, 90.7)
- moved C26 1.74 mm to (129.0, 98.2)
- moved R4 1.44 mm to (129.0, 96.4)
- moved SW1 1.06 mm to (120.3, 93.8)
- moved D3 0.71 mm to (99.9, 76.6)
- moved C43 0.65 mm to (88.7, 85.2)
- moved C45 0.56 mm to (94.1, 76.5)
- moved C44 0.54 mm to (96.9, 76.5)
- moved L1 0.47 mm to (94.7, 82.6)
- moved TP8 0.24 mm to (88.5, 81.9)
Routing:
- net +24V: track 179.4 -> 190.8 mm
- net +5V: track 20.5 -> 31.5 mm
- net /control/EN: track 0.00 -> 10.2 mm
- net +3.3V: track 19.8 -> 22.9 mm, vias 27 -> 32
- net Net-(LED5-A): track 0.00 -> 2.57 mm
- net /PowerSupply/vdc_in: track 25.9 -> 27.2 mm
- net Net-(C33-Pad1): track 12.2 -> 11.3 mm, vias 1 -> 0
- net GND: track 43.1 -> 43.7 mm, vias 66 -> 67

Commit message: FINISH TO DAY 17 JULY
COLOQUE TODAS LAS SALIDAS SOLO FALTA ROTEAR ALGUNAS COSAS AL ESP32
Parts:
- moved LED5 37.1 mm to (116.0, 94.8)
- moved R50 36.7 mm to (113.8, 94.8), turned to -90 degrees
- moved R26 8.62 mm to (130.8, 85.1), turned to 180 degrees
- moved R51 7.31 mm to (125.5, 123.9)
- moved C1 7.22 mm to (125.2, 116.7)
- moved C13 4.97 mm to (154.8, 100.4)
- moved C32 4.59 mm to (157.3, 100.4)
- moved C11 4.46 mm to (159.7, 100.4)
- moved U10 3.70 mm to (156.2, 105.2)
- moved C2 3.21 mm to (181.8, 109.4), turned to 180 degrees
- moved C15 2.92 mm to (152.0, 96.3)
- moved C19 2.42 mm to (132.5, 114.8), turned to 180 degrees
- moved C25 2.02 mm to (129.0, 101.7)
- moved C22 2.00 mm to (129.0, 99.9)
- moved TP5 1.89 mm to (184.4, 85.6)
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Routing:
- net /control/i2c_sda: track 0.00 -> 69.0 mm, vias 0 -> 4
- net /control/LED_INFO: track 0.00 -> 39.8 mm, vias 0 -> 2
- net /control/IN_NPN4: track 13.3 -> 48.7 mm, vias 0 -> 2
- net /control/IN-0-10V1/COM: track 2.90 -> 31.2 mm, vias 0 -> 2
- net /control/i2c_scl: track 0.00 -> 26.3 mm, vias 0 -> 2
- net +24V: track 190.8 -> 216.0 mm, vias 11 -> 16
- net /control/IN-0-10V/COM: track 2.57 -> 27.5 mm, vias 0 -> 2
- net /control/IN-0-10V/OUT3V: track 15.7 -> 39.7 mm, vias 0 -> 1
- net /control/OUT_RLY1: track 0.00 -> 19.2 mm
- net /control/IN_PNP1: track 3.39 -> 19.0 mm, vias 0 -> 2
- net GND: track 43.7 -> 56.8 mm, vias 67 -> 96
- net /control/EMRX: track 0.00 -> 11.3 mm
- net +3.3V: track 22.9 -> 33.9 mm, vias 32 -> 34
- net Net-(C21-Pad1): track 0.00 -> 8.34 mm
- net /control/OUT_RLY2: track 0.00 -> 8.31 mm, vias 0 -> 2
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
Commit message: update
Parts:
- moved TP9 1.05 mm to (183.7, 72.8)
- moved R54 0.49 mm to (166.9, 71.4)
- moved R53 0.49 mm to (170.8, 71.4)
- moved R58 0.28 mm to (187.1, 73.7)
- moved R27 0.16 mm to (157.7, 72.0)
- moved R9 0.14 mm to (155.4, 72.0)
- moved R14 0.06 mm to (146.5, 71.7)
- moved R44 0.06 mm to (152.6, 71.7)
Routing:
- net /control/IN-0-10V1/OUT3V: track 20.5 -> 36.6 mm
- net Net-(U16-RX/SDI): track 22.0 -> 15.0 mm
- net /control/IN-4-20MA1/OUT: track 4.38 -> 8.86 mm
- net /control/IN-4-20MA/OUT: track 6.99 -> 11.3 mm
- net /control/CON-IN_CT_P: track 6.51 -> 9.47 mm
- net GND: track 56.8 -> 59.5 mm, vias 96 -> 97
- net +3.3V: track 33.9 -> 33.4 mm

Commit message: UPDATE ESP32 RUTING
Routing:
- net /control/IN_NPN2: track 4.18 -> 48.4 mm, vias 0 -> 2
- net /control/IN_NPN3: track 3.68 -> 42.6 mm, vias 0 -> 2
- net /control/TEMP_CS: track 0.00 -> 37.3 mm, vias 0 -> 2
- net /control/EM_TX: track 8.05 -> 42.5 mm, vias 0 -> 2
- net /control/EMRX: track 11.3 -> 44.9 mm, vias 0 -> 2
- net /control/clk: track 0.00 -> 32.9 mm, vias 0 -> 2
- net /control/miso: track 0.00 -> 29.1 mm
- net /control/mosi: track 0.00 -> 27.9 mm
- net /control/IN_PNP2: track 3.97 -> 21.1 mm
- net GND: track 59.5 -> 60.5 mm
- net /control/i2c_sda: track 69.0 -> 69.9 mm
- net /control/i2c_scl: track 26.3 -> 27.1 mm
